File: kicad/1bit-cpu_asic.kicad_sch (KiCad schematic)
At the start: 46 parts, among them J1 USB_C_Receptacle_PowerOnly_6P, J2 Conn_01x11, Q1 2SC1815, Q2 2SC1815, Q3 2SC1815, SW1 SW, SW2 SW, SW3 SW_Push, U1 74HC04, U4 PTC06-1

Commit message: Fix U4's 20&21 pin.
Fix U4's 20&21 pin.
Connections:
- net +5V: now also U4.21 (VDD); no longer U4.20 (VSS)
- net GND: now also U4.20 (VSS); no longer U4.21 (VDD)
Changed lines of the file:
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@@
+	)
+	(junction
+		(at 215.9 78.74)
+		(diameter 0)
+		(color 0 0 0 0)
 	)
 	(junction
@@
 	)
 	(junction
+		(at 213.36 74.93)
+		(diameter 0)
+		(color 0 0 0 0)
+	)
+	(junction
 		(at 181.61 78.74)
 		(diameter 0)
@@
 	)
 	(junction
-		(at 213.36 78.74)
-		(diameter 0)
-		(color 0 0 0 0)
-	)
-	(junction
 		(at 167.64 128.27)
 		(diameter 0)
@@
 	(junction
 		(at 213.36 154.94)
-		(diameter 0)
-		(color 0 0 0 0)
-	)
-	(junction
-		(at 215.9 74.93)
 		(diameter 0)
 		(color 0 0 0 0)
@@
 	(wire
 		(pts
-			(xy 215.9 74.93) (xy 215.9 86.36)
+			(xy 215.9 72.39) (xy 215.9 78.74)
 		)
 		(stroke
@@
 	(wire
 		(pts
-			(xy 213.36 80.01) (xy 213.36 78.74)
+			(xy 213.36 19.05) (xy 213.36 74.93)
 		)
 		(stroke
@@
 	(wire
 		(pts
-			(xy 207.01 78.74) (xy 213.36 78.74)
-		)
-		(stroke
-			(width 0)
-			(type default)
-		)
-	)
-	(wire
-		(pts
 			(xy 107.95 106.68) (xy 110.49 106.68)
 		)
@@
 	(wire
 		(pts
+			(xy 210.82 74.93) (xy 213.36 74.93)
+		)
+		(stroke
+			(width 0)
+			(type default)
+		)
+	)
+	(wire
+		(pts
 			(xy 58.42 157.48) (xy 58.42 168.91)
 		)
@@
 	(wire
 		(pts
-			(xy 213.36 78.74) (xy 213.36 19.05)
-		)
-		(stroke
-			(width 0)
-			(type default)
-		)
-	)
-	(wire
-		(pts
 			(xy 52.07 92.71) (xy 52.07 118.11)
 		)
@@
 	(wire
 		(pts
+			(xy 215.9 78.74) (xy 215.9 86.36)
+		)
+		(stroke
+			(width 0)
+			(type default)
+		)
+	)
+	(wire
+		(pts
 			(xy 154.94 74.93) (xy 154.94 82.55)
 		)
@@
 	(wire
 		(pts
-			(xy 210.82 74.93) (xy 215.9 74.93)
-		)
-		(stroke
-			(width 0)
-			(type default)
-		)
-	)
-	(wire
-		(pts
-			(xy 275.59 81.28) (xy 166.37 81.28)
+			(xy 166.37 81.28) (xy 275.59 81.28)
 		)
 		(stroke
@@
 	(wire
 		(pts
+			(xy 213.36 74.93) (xy 213.36 80.01)
+		)
+		(stroke
+			(width 0)
+			(type default)
+		)
+	)
+	(wire
+		(pts
+			(xy 207.01 78.74) (xy 215.9 78.74)
+		)
+		(stroke
+			(width 0)
+			(type default)
+		)
+	)
+	(wire
+		(pts
 			(xy 33.02 90.17) (xy 163.83 90.17)
 		)
@@
 		)
 		(stroke
-			(width 0)
-			(type default)
-		)
-	)
-	(wire
-		(pts
-			(xy 215.9 72.39) (xy 215.9 74.93)
-		)
-		(stroke

Commit message: Fix U4's 40&41 pins.
Fix U4's 40&41 pins.
Connections:
- net +5V: now also U4.41 (VDD); no longer U4.40 (VSS)
- net GND: now also U4.40 (VSS); no longer U4.41 (VDD)
Changed lines of the file:
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@@
-	)
-	(junction
-		(at 210.82 19.05)
-		(diameter 0)
-		(color 0 0 0 0)
 	)
 	(junction
@@
 	)
 	(junction
+		(at 207.01 19.05)
+		(diameter 0)
+		(color 0 0 0 0)
+	)
+	(junction
 		(at 167.64 114.3)
 		(diameter 0)
@@
 	)
 	(junction
-		(at 215.9 22.86)
-		(diameter 0)
-		(color 0 0 0 0)
-	)
-	(junction
 		(at 261.62 45.72)
 		(diameter 0)
@@
 	(junction
 		(at 215.9 72.39)
+		(diameter 0)
+		(color 0 0 0 0)
+	)
+	(junction
+		(at 215.9 26.67)
 		(diameter 0)
 		(color 0 0 0 0)
@@
 	(wire
 		(pts
+			(xy 207.01 19.05) (xy 213.36 19.05)
+		)
+		(stroke
+			(width 0)
+			(type default)
+		)
+	)
+	(wire
+		(pts
 			(xy 142.24 101.6) (xy 142.24 130.81)
 		)
@@
 	(wire
 		(pts
-			(xy 215.9 21.59) (xy 215.9 22.86)
-		)
-		(stroke
-			(width 0)
-			(type default)
-		)
-	)
-	(wire
-		(pts
 			(xy 133.35 157.48) (xy 133.35 158.75)
 		)
@@
 	(wire
 		(pts
-			(xy 207.01 22.86) (xy 215.9 22.86)
-		)
-		(stroke
-			(width 0)
-			(type default)
-		)
-	)
-	(wire
-		(pts
 			(xy 236.22 146.05) (xy 236.22 144.78)
 		)
@@
 	(wire
 		(pts
-			(xy 213.36 19.05) (xy 210.82 19.05)
+			(xy 143.51 19.05) (xy 207.01 19.05)
 		)
 		(stroke
@@
 	(wire
 		(pts
-			(xy 210.82 19.05) (xy 143.51 19.05)
+			(xy 215.9 26.67) (xy 215.9 72.39)
 		)
 		(stroke
@@
 	(wire
 		(pts
+			(xy 210.82 26.67) (xy 215.9 26.67)
+		)
+		(stroke
+			(width 0)
+			(type default)
+		)
+	)
+	(wire
+		(pts
 			(xy 77.47 114.3) (xy 85.09 114.3)
 		)
@@
 	(wire
 		(pts
+			(xy 215.9 21.59) (xy 215.9 26.67)
+		)
+		(stroke
+			(width 0)
+			(type default)
+		)
+	)
+	(wire
+		(pts
 			(xy 144.78 157.48) (xy 144.78 158.75)
 		)
@@
 	(wire
 		(pts
-			(xy 215.9 22.86) (xy 215.9 72.39)
-		)
-		(stroke
-			(width 0)
-			(type default)
-		)
-	)
-	(wire
-		(pts
 			(xy 48.26 134.62) (xy 48.26 137.16)
 		)
@@
 	(wire
 		(pts
+			(xy 207.01 19.05) (xy 207.01 22.86)
+		)
+		(stroke
+			(width 0)
+			(type default)
+		)
+	)
+	(wire
+		(pts
 			(xy 107.95 106.68) (xy 110.49 106.68)
 		)
@@
 		)
 		(stroke
-			(width 0)
-			(type default)
-		)
-	)
-	(wire
-		(pts
-			(xy 210.82 26.67) (xy 210.82 19.05)
-		)
-		(stroke
